Commit message: clearning of apc_config

File: catkin_ws/src/apc_config/models/IRB1600ID/irb_1600id.urdf (robot description, URDF)
Before this commit: robot irb_1600id, 14 links, 13 joints
Links:
- removed link finger_left
- removed link finger_right
- removed link gripper_left
- removed link gripper_right
- added link bot_finger; visual mesh filename=package://apc_config/models/wsg_50/meshes/arc2017/bot_finge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 scale=0.001 0.001 0.001
- added link bot_spatula_centered; visual mesh filename=package://apc_config/models/wsg_50/meshes/arc2017/bot_spatu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 scale=0.001 0.001 0.001
- added link top_finger; visual mesh filename=package://apc_config/models/wsg_50/meshes/arc2017/top_finge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 scale=0.001 0.001 0.001
- added link top_spatula; visual mesh filename=package://apc_config/models/wsg_50/meshes/arc2017/top_spatu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 scale=0.001 0.001 0.001
- link base_link: mass 6.21503193527 -> None; geometry visual mesh filename=package://apc_config/models/IRB1600ID/meshes/visual/base_li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
- link hand_mount: mass 0.0258654328719498 -> None
- link link_1: mass 16.287755696602 -> None; geometry visual mesh filename=package://apc_config/models/IRB1600ID/meshes/visual/link_1.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
- link link_2: mass 7.58037424484438 -> None; geometry visual mesh filename=package://apc_config/models/IRB1600ID/meshes/visual/link_2.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
- link link_3: mass 8.03072730997701 -> None; geometry visual mesh filename=package://apc_config/models/IRB1600ID/meshes/visual/link_3.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
- link link_4: mass 1.7702548022269 -> None; geometry visual mesh filename=package://apc_config/models/IRB1600ID/meshes/visual/link_4.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
- link link_5: mass 0.145550520315438 -> None; geometry visual mesh filename=package://apc_config/models/IRB1600ID/meshes/visual/link_5.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
- link link_6: mass 0.0258654328719498 -> None; geometry visual mesh filename=package://apc_config/models/IRB1600ID/meshes/visual/link_6.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
- link link_wrist: mass 0.0258654328719498 -> None; geometry visual mesh filename=package://apc_config/models/wsg_50/meshes/arc2017/wrist_bod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 scale=0.001 0.001 0.001
- link wsg50_base_link: mass 1.2 -> None; geometry visual mesh filename=package://apc_config/models/wsg_50/meshes/arc2017/gripper_c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 scale=0.001 0.001 0.001
Joints:
- removed joint guide_joint_finger_left
- removed joint guide_joint_finger_right
- added joint bot_spatula_joint: type revolute, parent bot_finger, child bot_spatula_centered, origin xyz=0.00730000 0 .367279 rpy=0 0 0, axis 0 1 0, limit lower=-.4 upper=0 effort=1 velocity=1
- added joint top_spatula_joint: type fixed, parent top_finger, child top_spatula, origin xyz=0 0 0 rpy=0 0 0, axis -1 0 0
- joint joint7: axis 0 0 1 -> 0 1 0; limit lower=-6.98131700798 upper=6.981317007989 effort=300 velocity=7.33 -> lower=-3.49065850399 upper=3.49065850399 effort=300 velocity=7.33
- joint joint_hand: axis 0 0 1 -> (none); parent hand_mount -> link_wrist
- joint wsg_50_gripper_base_joint_gripper_left: child gripper_left -> top_finger; limit lower=-0.055 upper=-0.0027 effort=1.0 velocity=1.0 -> lower=-0.055 upper=0 effort=1.0 velocity=1.0; parent wsg50_base_link -> link_wrist
- joint wsg_50_gripper_base_joint_gripper_right: axis -1 0 0 -> 1 0 0; child gripper_right -> bot_finger; limit lower=0.0027 upper=0.055 effort=1.0 velocity=1.0 -> lower=0 upper=0.055 effort=1.0 velocity=1.0; origin xyz=0 0 0 rpy=0 0 3.14159 -> xyz=0 0 0 rpy=0 0 0; parent wsg50_base_link -> link_wrist
